File: doc/kicad/WeatherStation.kicad_pcb (KiCad board)
At the start: 4 copper layers, 88.9 x 68.6 mm, 22 parts, among them J10 Screw_Terminal_01x04, J11 Screw_Terminal_01x02, J15 Screw_Terminal_01x02, J16 Conn_01x02_Male, J8 Screw_Terminal_01x04, J9 Screw_Terminal_01x02, Q1 IRLML2244, SW1 Reset, SW2 Mode, U4 Rain_Sensor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

Commit message: Stable without Solar monitor
Parts:
- added J19: Prog, Socket_Strips:Socket_Strip_Straight_1x06_Pitch2.54mm, F.Cu at (192.4, 75.6)
Routing:
- net /RST: track 14.1 -> 52.5 mm
- net GND: track 339.3 -> 360.2 mm
- net /PROG: track 46.1 -> 54.8 mm
- net /TxD: track 0.00 -> 4.44 mm
- net /RxD: track 0.00 -> 4.44 mm
Changed lines of the file:
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@@
     (thickness 1.6)
     (drawings 4)
-    (tracks 173)
+    (tracks 186)
     (zones 0)
-    (modules 22)
-    (nets 53)
+    (modules 23)
+    (nets 54)
   )
   (page A4)
@@
   )
   (setup
-    (last_trace_width 0.25)
+    (last_trace_width 0.5)
     (user_trace_width 0.5)
     (user_trace_width 1)
@@
   (net 51 "Net-(U7-Pad6)")
   (net 52 "Net-(U7-Pad3)")
+  (net 53 "Net-(J19-Pad4)")
   (net_class Default "Dies ist die voreingestellte Netzklasse."
     (clearance 0.2)
@@
     (add_net "Net-(J15-Pad1)")
     (add_net "Net-(J16-Pad2)")
+    (add_net "Net-(J19-Pad4)")
     (add_net "Net-(J9-Pad1)")
     (add_net "Net-(Q1-Pad1)")
@@
     (pad 10 thru_hole circle (at 2.54 -5.08 90) (size 1.524 1.524) (drill 0.762) (layers *.Cu *.Mask))
   )
+  (module Socket_Strips:Socket_Strip_Straight_1x06_Pitch2.54mm (layer F.Cu)
+    (at 192.405 75.565)
+    (descr "Through hole straight socket strip, 1x06, 2.54mm pitch, single row")
+    (tags "Through hole socket strip THT 1x06 2.54mm single row")
+    (fp_text reference J19 (at 0 -2.33) (layer F.SilkS)
+      (effects (font (size 1 1) (thickness 0.15)))
+    )
+    (fp_text value Prog (at 0 15.03) (layer F.Fab)
+      (effects (font (size 1 1) (thickness 0.15)))
+    )
+    (fp_text user %R (at 0 -2.33) (layer F.Fab)
+      (effects (font (size 1 1) (thickness 0.15)))
+    )
+    (fp_line (start 1.8 -1.8) (end -1.8 -1.8) (layer F.CrtYd) (width 0.05))
+    (fp_line (start 1.8 14.5) (end 1.8 -1.8) (layer F.CrtYd) (width 0.05))
+    (fp_line (start -1.8 14.5) (end 1.8 14.5) (layer F.CrtYd) (width 0.05))
+    (fp_line (start -1.8 -1.8) (end -1.8 14.5) (layer F.CrtYd) (width 0.05))
+    (fp_line (start -1.33 -1.33) (end 0 -1.33) (layer F.SilkS) (width 0.12))
+    (fp_line (start -1.33 0) (end -1.33 -1.33) (layer F.SilkS) (width 0.12))
+    (fp_line (start 1.33 1.27) (end -1.33 1.27) (layer F.SilkS) (width 0.12))
+    (fp_line (start 1.33 14.03) (end 1.33 1.27) (layer F.SilkS) (width 0.12))
+    (fp_line (start -1.33 14.03) (end 1.33 14.03) (layer F.SilkS) (width 0.12))
+    (fp_line (start -1.33 1.27) (end -1.33 14.03) (layer F.SilkS) (width 0.12))
+    (fp_line (start 1.27 -1.27) (end -1.27 -1.27) (layer F.Fab) (width 0.1))
+    (fp_line (start 1.27 13.97) (end 1.27 -1.27) (layer F.Fab) (width 0.1))
+    (fp_line (start -1.27 13.97) (end 1.27 13.97) (layer F.Fab) (width 0.1))
+    (fp_line (start -1.27 -1.27) (end -1.27 13.97) (layer F.Fab) (width 0.1))
+    (pad 6 thru_hole oval (at 0 12.7) (size 1.7 1.7) (drill 1) (layers *.Cu *.Mask)
+      (net 2 GND))
+    (pad 5 thru_hole oval (at 0 10.16) (size 1.7 1.7) (drill 1) (layers *.Cu *.Mask)
+      (net 15 /PROG))
+    (pad 4 thru_hole oval (at 0 7.62) (size 1.7 1.7) (drill 1) (layers *.Cu *.Mask)
+      (net 53 "Net-(J19-Pad4)"))
+    (pad 3 thru_hole oval (at 0 5.08) (size 1.7 1.7) (drill 1) (layers *.Cu *.Mask)
+      (net 43 /RxD))
+    (pad 2 thru_hole oval (at 0 2.54) (size 1.7 1.7) (drill 1) (layers *.Cu *.Mask)
+      (net 44 /TxD))
+    (pad 1 thru_hole rect (at 0 0) (size 1.7 1.7) (drill 1) (layers *.Cu *.Mask)
+      (net 1 /RST))
+    (model ${KISYS3DMOD}/Socket_Strips.3dshapes/Socket_Strip_Straight_1x06_Pitch2.54mm.wrl
+      (offset (xyz 0 -6.349999904632568 0))
+      (scale (xyz 1 1 1))
+      (rotate (xyz 0 0 270))
+    )
+  )
   (gr_line (start 127 62.865) (end 215.9 62.865) (layer Edge.Cuts) (width 0.1))
   (gr_line (start 215.9 131.445) (end 215.9 62.865) (layer Edge.Cuts) (width 0.1))
@@
   (segment (start 144.24 73.025) (end 143.66 72.445) (width 0.5) (layer B.Cu) (net 1) (status 30))
   (segment (start 147.32 73.025) (end 144.24 73.025) (width 0.5) (layer B.Cu) (net 1) (status 20))
+  (segment (start 191.055 75.565) (end 192.405 75.565) (width 0.5) (layer B.Cu) (net 1))
+  (segment (start 189.842999 76.777001) (end 191.055 75.565) (width 0.5) (layer B.Cu) (net 1))
+  (segment (start 156.152001 76.777001) (end 189.842999 76.777001) (width 0.5) (layer B.Cu) (net 1))
+  (segment (start 154.94 75.565) (end 156.152001 76.777001) (width 0.5) (layer B.Cu) (net 1))
   (segment (start 208.28 126.365) (end 208.28 128.905) (width 0.5) (layer B.Cu) (net 2) (status 10))
   (segment (start 207.24 100.965) (end 208.28 100.965) (width 0.5) (layer B.Cu) (net 2) (status 10))
@@
   (segment (start 213.36 100.965) (end 213.36 97.155) (width 0.5) (layer B.Cu) (net 2))
   (segment (start 208.28 84.225) (end 207.24 83.185) (width 0.5) (layer B.Cu) (net 2))
-  (segment (start 208.28 100.965) (end 208.28 84.225) (width 0.5) (layer B.Cu) (net 2))
+  (segment (start 192.405 93.345) (end 208.28 93.345) (width 0.5) (layer B.Cu) (net 2))
+  (segment (start 192.405 88.265) (end 192.405 93.345) (width 0.5) (layer B.Cu) (net 2))
+  (segment (start 208.28 100.965) (end 208.28 93.345) (width 0.5) (layer B.Cu) (net 2))
+  (segment (start 208.28 93.345) (end 208.28 84.225) (width 0.5) (layer B.Cu) (net 2))
   (via (at 203.2 106.045) (size 0.8) (drill 0.4) (layers F.Cu B.Cu) (net 3))
   (segment (start 202.25 108.585) (end 202.25 106.995) (width 0.5) (layer F.Cu) (net 3) (status 10))
@@
   (segment (start 198.12 100.965) (end 200.66 98.425) (width 0.5) (layer In1.Cu) (net 15))
   (segment (start 200.66 74.145) (end 201.78 73.025) (width 0.5) (layer In1.Cu) (net 15) (status 20))
-  (segment (start 200.66 98.425) (end 200.66 74.145) (width 0.5) (layer In1.Cu) (net 15))
+  (segment (start 200.444999 84.874999) (end 200.66 85.09) (width 0.5) (layer In1.Cu) (net 15))
+  (segment (start 193.255001 84.874999) (end 200.444999 84.874999) (width 0.5) (layer In1.Cu) (net 15))
+  (segment (start 192.405 85.725) (end 193.255001 84.874999) (width 0.5) (layer In1.Cu) (net 15))
+  (segment (start 200.66 98.425) (end 200.66 85.09) (width 0.5) (layer In1.Cu) (net 15))
+  (segment (start 200.66 85.09) (end 200.66 74.145) (width 0.5) (layer In1.Cu) (net 15))
   (via (at 203.2 113.665) (size 0.8) (drill 0.4) (layers F.Cu B.Cu) (net 16))
   (segment (start 203.2 110.585) (end 203.2 113.665) (width 0.5) (layer F.Cu) (net 16) (status 10))
@@
   (segment (start 172.72 108.585) (end 173.932001 107.372999) (width 0.5) (layer In1.Cu) (net 21))
   (segment (start 173.932001 107.372999) (end 173.932001 97.843239) (width 0.5) (layer In1.Cu) (net 21))
+  (segment (start 187.96 80.645) (end 192.405 80.645) (width 0.5) (layer B.Cu) (net 43))
+  (segment (start 187.96 78.105) (end 192.405 78.105) (width 0.5) (layer B.Cu) (net 44))
 )
